File: RippleCounters/Counters.sch (KiCad schematic (older format))
At the start: 4 parts

Commit message: add sync counter HW
Parts:
- added C? (x2): C_small, symbol 00TJR:C_small
- added D? (x4): LED, symbol 00TJR:LED
- added R? (x3): R, symbol 00TJR:R
- added R? (x4): 330, symbol 00TJR:R
- added U? (x12): 7476, symbol 74xx:74LS76
- added U? (x13): 74LS08, symbol 74xx:74LS08
- added U? (x9): 74LS04, symbol 74xx:74LS04
Connections:
- net Clock: now reaches U?.1
- net Clock: now also U?.1, U?.1, U?.1, U?.1, U?.1, U?.1, U?.1, U?.1, U?.1
- net ~Q0: now reaches U?.14
- net ~Q0: now also R?.1
- net Q0: now reaches U?.15 (Q)
- net Q0: now also U?.6
- net VCC: now reaches U?.16 (K)
- net VCC: now also U?.12 (K), U?.12 (K), U?.16 (K), U?.2, U?.2, U?.4 (J), U?.4 (J), U?.7, U?.7, U?.9 (J), U?.9 (J), D?.2 (A), D?.2 (A), D?.2 (A), D?.2 (A), R?.1, R?.1, U?.16 (K), U?.16 (K), U?.16 (K), U?.16 (K), U?.16 (K), U?.2, U?.2, U?.2, U?.2, U?.2, U?.2, U?.2, U?.2, U?.4 (J), U?.4 (J), U?.4 (J), U?.4 (J), U?.4 (J)
- net ~Reset: now reaches U?.3
- net ~Reset: now also U?.3, U?.8, U?.8
- net Q1: now reaches U?.1
- net Q1: now also U?.11 (Q)
- net ~Q2: now reaches U?.14
- net ~Q2: now also R?.1
- net Q2: now reaches U?.15 (Q)
- net Q2: now also U?.6
- new net: D?.1 (K), R?.2 (x4)
- new net: U?.1, U?.1, U?.15 (Q) (x3)
- new net: U?.3, U?.3, U?.3, U?.3, U?.3 (x2)
- new net: U?.1, U?.15 (Q)
- new net: C?.1, R?.2, U?.1 (x2)
- new net: U?.2, U?.2 (x6)
- new net: U?.2, U?.3 (x3)
- new net: U?.1, U?.3 (x5)
- new net: U?.1, U?.1, U?.15 (Q), U?.16 (K), U?.4 (J)
- new net: U?.15 (Q), U?.2, U?.2
- new net: U?.1, U?.15 (Q), U?.2
- new net: U?.1, U?.16 (K), U?.3, U?.4 (J)
- new net: U?.15 (Q), U?.2
- new net: U?.16 (K), U?.3, U?.4 (J)
- new net: U?.1, U?.2 (x3)
- new net GND: C?.2, C?.2
- new net Q3: U?.11 (Q)
- new net ~Q1: R?.1, U?.10
- new net ~Q3: R?.1, U?.10
- no-connect marks 0 -> 8
